File: Armement2026.kicad_sch (KiCad schematic)
At the start: 24 parts, among them J1 Screw_Terminal_01x02, J10 Screw_Terminal_01x02, J11 Screw_Terminal_01x02, J12 Screw_Terminal_01x02, J2 Screw_Terminal_01x02, J5 Screw_Terminal_01x02, J6 Screw_Terminal_01x02, J8 Screw_Terminal_01x02, J9 Screw_Terminal_01x02, Q1 NTR4101PT1G, Q2 NTR4101PT1G, SW1 SW_Nidec_CAS-120A1, SW2 SW_Nidec_CAS-120A1, SW3 SW_Nidec_CAS-120A1, U1 LDO_4v2-MIC5209-4.2YS-TR

Commit message: PCB Armement IRECxFAR-OUT
Parts:
- removed F1: Polyfuse, Fuse:Fuse_1812_4532Metric, symbol Device:Polyfuse
- removed J10: Screw_Terminal_01x02, Connector_PinHeader_2.54mm:PinHeader_1x02_P2.54mm_Vertical, symbol Connector:Screw_Terminal_01x02
- removed J12: Screw_Terminal_01x02, Connector_Molex:Molex_Micro-Fit_3.0_43650-0215_1x02_P3.00mm_Vertical, symbol Connector:Screw_Terminal_01x02
- removed J9: Screw_Terminal_01x02, Connector_PinHeader_1.27mm:PinHeader_1x02_P1.27mm_Vertical, symbol Connector:Screw_Terminal_01x02
- added J3, J4: Screw_Terminal_01x02, Connector_AMASS:AMASS_XT30U-M_1x02_P5.0mm_Vertical, symbol Connector:Screw_Terminal_01x02
- added J7: Screw_Terminal_01x02, Connector_JST:JST_SH_BM02B-SRSS-TB_1x02-1MP_P1.00mm_Vertical, symbol Connector:Screw_Terminal_01x02
- added JP1, JP2, JP3, JP4, JP5: SolderJumper_2_Open, Jumper:SolderJumper-2_P1.3mm_Open_TrianglePad1.0x1.5mm, symbol Jumper:SolderJumper_2_Open
- C1, C2, C7, C8: Digikey_Part_Number (none) -> 1276-1097-1-ND - Cut Tape (CT); Manufacture_Part_Number (none) -> CL31B105KAHNNNE
- DZ1, DZ2: Digikey_Part_Number (none) -> SZMMSZ4679T1GOSCT-ND - Cut Tape (CT); Manufacture_Part_Number (none) -> SZMMSZ4679T1G
- J1: Digikey_Part_Number (none) -> 1738-1437-ND; Manufacture_Part_Number (none) -> FIT0587
- J11: Digikey_Part_Number (none) -> 1738-1436-ND; Manufacture_Part_Number (none) -> FIT0586
- J2: footprint footprints:CONN_70545-xxxx_02_MOL -> Connector_Molex:Molex_Micro-Fit_3.0_43650-0215_1x02_P3.00mm_Vertical; Digikey_Part_Number (none) -> WM1860-ND; Fem Con (none) -> https://www.digikey.ca/en/products/detail/molex/2147551021/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; Manufacture_Part_Number (none) -> 0436500200
- J5: footprint 3mm header 2x1:CONN_SD-44067-001_02_MOL -> Connector_AMASS:AMASS_XT30U-M_1x02_P5.0mm_Vertical; Digikey_Part_Number (none) -> 1738-1436-ND; LCSC Part # (none) -> C129184; Manufacture_Part_Number (none) -> FIT0586
- J6: footprint footprints:CONN_SDA_43255-00XX_02_MOL -> footprints:CONN_70545-xxxx_02_MOL; Digikey_Part_Number (none) -> 23-0705450001-ND; Fem Con (none) -> https://www.digikey.ca/en/products/detail/molex/0015388020/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; Manufacture_Part_Number (none) -> 0705450001
- J8: footprint footprints:CONN02_560020_MOL -> Connector_JST:JST_PH_B2B-PH-K_1x02_P2.00mm_Vertical; Digikey_Part_Number (none) -> 455-1704-ND; Fem Con (none) -> https://www.digikey.ca/en/products/detail/jst-sales-america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; Manufacture_Part_Number (none) -> B2B-PH-K-S
- PWR_R1, PWR_R2: Digikey_Part_Number (none) -> 541-100KUCT-ND - Cut Tape (CT); Manufacture_Part_Number (none) -> CRCW1206100KFKEAHP
- Q1, Q2: Digikey_Part_Number (none) -> NTR4101PT1GOSCT-ND - Cut Tape (CT); Manufacture_Part_Number (none) -> NTR4101PT1G
- SW1, SW2, SW3: Digikey_Part_Number (none) -> SW871-ND; Manufacture_Part_Number (none) -> SS-5GL13
- U1: Digikey_Part_Number (none) -> MIC5209-4.2YS-CT-ND - Cut Tape (CT); Manufacture_Part_Number (none) -> MIC5209-4.2YS-TR
Connections:
- net 7v4: now also DZ1.1 (K), Q1.3 (S), J3.2 (Pin_2), J4.2 (Pin_2), JP2.2 (B), JP3.2 (B); no longer J5.1 (Pin_1), J6.1 (Pin_1), J8.1 (Pin_1)
- net GND: now also J5.1 (Pin_1), J3.1 (Pin_1), J4.1 (Pin_1); no longer J1.1 (Pin_1), J5.2 (Pin_2), J6.2 (Pin_2), Q1.1 (D), SW1.1 (C), SW1.2 (B)
- net at C7.1, DZ2.1 (K), Q2.3 (S): now also J2.1 (Pin_1)
- net at C7.2, PWR_R2.2: now also J2.2 (Pin_2), J6.1 (Pin_1), JP1.1 (A)
- net at SW3.2 (B): now also J6.2 (Pin_2)
- net at C2.1, U1.3 (OUT): now also J8.1 (Pin_1)
- net at SW2.1 (C): now also J7.1 (Pin_1), JP5.1 (A); no longer J2.1 (Pin_1)
- net at SW2.2 (B): now also JP3.1 (A), JP4.1 (A); no longer J2.2 (Pin_2)
- net at Q2.1 (D), SW3.1 (C): now also JP1.2 (B)
- new net: J1.1 (Pin_1), SW1.1 (C)
- new net: J5.2 (Pin_2), JP2.1 (A), JP5.2 (B)
- new net: J7.2 (Pin_2), JP4.2 (B)
- new net: Q1.1 (D), SW1.2 (B)
Other:
- note added: "1"
- note added: "2"
- note added: "Si on veut l'ODB sur sa propre switch comme à l'IREC, on peut souder les 2 Si on veut que ce soit le stratologger et que l'ODB soit avec les autres composantes comme à Far-out, on soude 1"
- moved on the sheet: C7, DZ2, PWR_R2, Q2
