File: Armement2026.kicad_sch (KiCad schematic)
At the start: 31 parts, among them J1 Screw_Terminal_01x02, J10 Screw_Terminal_01x02, J11 Screw_Terminal_01x02, J2 Screw_Terminal_01x02, J3 Screw_Terminal_01x02, J4 Screw_Terminal_01x02, J5 Screw_Terminal_01x02, J6 Screw_Terminal_01x02, J7 Screw_Terminal_01x02, J8 Screw_Terminal_01x02, J9 Screw_Terminal_01x02, Q1 NTR4101PT1G, Q2 NTR4101PT1G, SW1 SW_Nidec_CAS-120A1, SW2 SW_Nidec_CAS-120A1, SW3 SW_Nidec_CAS-120A1, SW4 SW_Nidec_CAS-120A1, U1 LDO_4v2-MIC5209-4.2YS-TR

Commit message: wtf did I just do
Parts:
- added J12: Screw_Terminal_01x02, TerminalBlock:TerminalBlock_MaiXu_MX126-5.0-02P_1x02_P5.00mm, symbol Connector:Screw_Terminal_01x02
- added JP6: SolderJumper_2_Open, Jumper:SolderJumper-2_P1.3mm_Open_TrianglePad1.0x1.5mm, symbol Jumper:SolderJumper_2_Open
- J2: footprint Connector_Molex:Molex_Micro-Fit_3.0_43650-0215_1x02_P3.00mm_Vertical -> 3mm header 2x1:CONN_SD-44067-001_02_MOL
- J7: footprint Connector_JST:JST_SH_BM02B-SRSS-TB_1x02-1MP_P1.00mm_Vertical -> Connector_PinHeader_2.54mm:PinHeader_1x02_P2.54mm_Vertical; Digikey_Part_Number 455-1788-1-ND - Cut Tape (CT) -> WM2700-ND; Fem Con https://www.digikey.ca/en/products/detail/jst-sales-america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 -> (none); Manufacture_Part_Number BM02B-SRSS-TB -> 0022112022; wire (none) -> https://www.digikey.ca/en/products/detail/molex/2177971021/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
- J9: footprint RCJ_054:CUI_RCJ-054 -> Connector_JST:JST_SH_BM02B-SRSS-TB_1x02-1MP_P1.00mm_Vertical; Digikey_Part_Number CP-1427-ND -> 455-1788-1-ND - Cut Tape (CT); Fem Con (none) -> https://www.digikey.ca/en/products/detail/jst-sales-america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; Manufacture_Part_Number RCJ-054 -> BM02B-SRSS-TB
- Q1: value NTR4101PT1G -> DMP10H400SK3-13; footprint NTR4101PT1G:SOT-23-3_1P4X3P040_ONS -> footprints3:TO252-DPAK-DMP10H400SK3_DIO; Digikey NTR4101PT1GOSCT-ND -> DMP10H400SK3-13; Digikey_Part_Number NTR4101PT1GOSCT-ND - Cut Tape (CT) -> DMP10H400SK3-13DICT-ND - Cut Tape (CT); Manufacture_Part_Number NTR4101PT1G -> DMP10H400SK3-13
- Q2: value NTR4101PT1G -> DMP10H400SK3-13; footprint NTR4101PT1G:SOT-23-3_1P4X3P040_ONS -> footprints3:TO252-DPAK-DMP10H400SK3_DIO; Digikey NTR4101PT1GOSCT-ND -> DMP10H400SK3-13; Digikey_Part_Number NTR4101PT1GOSCT-ND - Cut Tape (CT) -> DMP10H400SK3-13DICT-ND; Manufacture_Part_Number NTR4101PT1G -> DMP10H400SK3-13
Connections:
- net 7v4: now also J5.2 (Pin_2); no longer C1.1, JP3.2 (B), U1.1 (IN)
- net GND: now also JP5.1 (A)
- net at J10.1 (Pin_1), SW4.3 (A): now also J12.2 (Pin_2); no longer J9.2 (Pin_2)
- net at J10.2 (Pin_2), SW4.1 (C): now also JP4.1 (A)
- net at C2.1, J8.1 (Pin_1), U1.3 (OUT): now also JP3.2 (B)
- net at C7.2, J2.2 (Pin_2), JP1.1 (A)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: now also J6.2 (Pin_2); no longer J6.1 (Pin_1)
- net at J7.2 (Pin_2): now also SW2.2 (B); no longer JP4.2 (B)
- net at J9.1 (Pin_1): now also JP4.2 (B); no longer SW4.2 (B)
- net at SW3.2 (B): now also J6.1 (Pin_1); no longer J6.2 (Pin_2)
- new net: JP5.2 (B), JP6.1 (A), SW2.1 (C)
- new net: J7.1 (Pin_1), JP3.1 (A), JP6.2 (B)
- new net: J12.1 (Pin_1), J9.2 (Pin_2), SW4.2 (B)
- new net: C1.1, JP2.1 (A), U1.1 (IN)
Other:
- note added: "3"
- note added: "Batterie featherweigth x strato"
- note added: "On soude 1 si on veut le strato, sinon on a le shunt motor"
- note added: "On soude 2, on va avoir le strato sur une switch et le featherweigth avec tout le reste du système"
- note added: "On soude 3 si on veut le featherweigth sur sa propre switch"
- note added: "Stratologger x"
- note added: "x Easymini"
- note removed: "Si on veut l'ODB sur sa propre switch comme à l'IREC, on peut souder les 2 Si on veut que ce soit le stratologger et que l'ODB soit avec les autres composantes comme à Far-out, on soude 1"
- note removed: "Stratologger"
- moved on the sheet: C1, C2, J8, U1
