File: BMS 2S/BMS 2S.kicad_sch (KiCad schematic)
At the start: 24 parts, among them J1 Screw_Terminal_01x01, J2 Screw_Terminal_01x01, J3 Screw_Terminal_01x01, J4 Screw_Terminal_01x01, J5 Screw_Terminal_01x01, J6 Screw_Terminal_01x01, Q1 ZXMN4A06K, Q2 ZXMN4A06K, Q3 DMG2302UK-7, Q4 DMG2302UK-7, U1 S-8252AAZ-M6T1U, U2 S-8252AAZ-M6T1U

Commit message: commande pcbway
Parts:
- J1, J2, J3, J4, J5, J6: Digikey_Part_Number (none) -> -; Manufacturer_Product_Number (none) -> -
- OUT2: Digikey_Part_Number (none) -> 23-0705450001-ND; Manufacturer_Product_Number (none) -> 0705450001

Commit message: Bom du bms
Parts:
- C1, C2, C3, C4: Digikey_Part_Number (none) -> 399-C1206C104J5RACTUCT-ND; Manufacturer_Product_Number (none) -> C1206C104J5RACTU
- OUT1: Digikey_Part_Number (none) -> 1738-1437-ND; Manufacturer_Product_Number (none) -> FIT0587
- Q1: Digikey_Part_Number (none) -> 31-ZXMN4A06KTCCT-ND; Manufacturer_Product_Number (none) -> ZXMN4A06KTC
- Q2: footprint BMS_footprints:SOT23_DMG230_DIO -> TO-252-2; Digikey_Part_Number (none) -> 31-ZXMN4A06KTCCT-ND; Manufacturer_Product_Number (none) -> ZXMN4A06KTC
- Q3, Q4: Digikey_Part_Number (none) -> DMG2302UK-7DICT-ND; Manufacturer_Product_Number (none) -> DMG2302UK-7
- R1, R2, R4, R5: Digikey_Part_Number (none) -> 311-470FRCT-ND; Manufacturer_Product_Number (none) -> RC1206FR-07470RL
- R3, R6: Digikey_Part_Number (none) -> 738-RMCF1206FG2K00CT-ND; Manufacturer_Product_Number (none) -> RMCF1206FG2K00
- U1, U2: Digikey_Part_Number (none) -> 1662-S-8252AAG-M6T1UCT-ND; Manufacturer_Product_Number (none) -> S-8252AAG-M6T1U
Changed lines of the file:
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@@
 			)
 		)
-		(property "Datasheet" "https://www.diodes.com/assets/Datasheets/ZXMN4A06K.pdf"
+		(property "Datasheet" "https://www.digikey.ca/en/products/detail/diodes-incorporated/ZXMN4A06KTC/991923?s=N4IgTCBcDaIFoA0CyA5ALAQQAwDYDSIAugL5A"
 			(at 121.92 106.68 0)
 			(effects
@@
 			)
 		)
-		(property "Digikey_Part_Number" ""
+		(property "Digikey_Part_Number" "31-ZXMN4A06KTCCT-ND"
 			(at 121.92 106.68 0)
 			(effects
@@
 			)
 		)
-		(property "Manufacturer_Product_Number" ""
+		(property "Manufacturer_Product_Number" "  ZXMN4A06KTC"
 			(at 121.92 106.68 0)
 			(effects
@@
 			)
 		)
-		(property "Datasheet" "~"
+		(property "Datasheet" "https://www.digikey.ca/en/products/detail/stackpole-electronics-inc/RMCF1206FG2K00/1758859"
 			(at 123.19 73.66 0)
 			(effects
@@
 			)
 		)
-		(property "Digikey_Part_Number" ""
+		(property "Digikey_Part_Number" "738-RMCF1206FG2K00CT-ND"
 			(at 123.19 73.66 90)
 			(effects
@@
 			)
 		)
-		(property "Manufacturer_Product_Number" ""
+		(property "Manufacturer_Product_Number" "RMCF1206FG2K00"
 			(at 123.19 73.66 90)
 			(effects
@@
 			)
 		)
-		(property "Datasheet" "~"
+		(property "Datasheet" "https://www.digikey.ca/en/products/detail/yageo/RC1206FR-07470RL/728934"
 			(at 53.34 93.98 0)
 			(effects
@@
 			)
 		)
-		(property "Digikey_Part_Number" ""
+		(property "Digikey_Part_Number" "311-470FRCT-ND"
 			(at 53.34 93.98 90)
 			(effects
@@
 			)
 		)
-		(property "Manufacturer_Product_Number" ""
+		(property "Manufacturer_Product_Number" "RC1206FR-07470RL"
 			(at 53.34 93.98 90)
 			(effects
@@
 			)
 		)
-		(property "Datasheet" "~"
+		(property "Datasheet" "https://www.digikey.ca/en/products/detail/dfrobot/FIT0587/9559256"
 			(at 88.9 48.26 0)
 			(effects
@@
 			)
 		)
-		(property "Digikey_Part_Number" ""
+		(property "Digikey_Part_Number" "1738-1437-ND"
 			(at 88.9 48.26 0)
 			(effects
@@
 			)
 		)
-		(property "Manufacturer_Product_Number" ""
+		(property "Manufacturer_Product_Number" "FIT0587"
 			(at 88.9 48.26 0)
 			(effects
@@
 			)
 		)
-		(property "Datasheet" "~"
+		(property "Datasheet" "https://www.digikey.ca/en/products/detail/kemet/C1206C104J5RACTU/411249"
 			(at 59.69 105.41 0)
 			(effects
@@
 			)
 		)
-		(property "Digikey_Part_Number" ""
+		(property "Digikey_Part_Number" "399-C1206C104J5RACTUCT-ND"
 			(at 59.69 105.41 0)
 			(effects
@@
 			)
 		)
-		(property "Manufacturer_Product_Number" ""
+		(property "Manufacturer_Product_Number" "C1206C104J5RACTU"
 			(at 59.69 105.41 0)
 			(effects
@@
 			)
 		)
-		(property "Digikey_Part_Number" ""
+		(property "Digikey_Part_Number" "1662-S-8252AAG-M6T1UCT-ND"
 			(at 115.57 96.52 0)
 			(effects
@@
 			)
 		)
-		(property "Manufacturer_Product_Number" ""
+		(property "Manufacturer_Product_Number" "S-8252AAG-M6T1U"
 			(at 115.57 96.52 0)
 			(effects
@@
 			)
 		)
-		(property "Datasheet" "~"
+		(property "Datasheet" "https://www.digikey.ca/en/products/detail/stackpole-electronics-inc/RMCF1206FG2K00/1758859"
 			(at 240.03 69.85 0)
 			(effects
@@
 			)
 		)
-		(property "Digikey_Part_Number" ""
+		(property "Digikey_Part_Number" "738-RMCF1206FG2K00CT-ND"
 			(at 240.03 69.85 90)
 			(effects
@@
 			)
 		)
-		(property "Manufacturer_Product_Number" ""
+		(property "Manufacturer_Product_Number" "RMCF1206FG2K00"
 			(at 240.03 69.85 90)
 			(effects
@@
 			)
 		)
-		(property "Datasheet" "https://www.diodes.com/assets/Datasheets/DMG2302UK.pdf"
+		(property "Datasheet" "https://www.digikey.ca/en/products/detail/diodes-incorporated/DMG2302UK-7/6010142"
 			(at 238.76 102.87 0)
 			(effects
@@
 			)
 		)
-		(property "Digikey_Part_Number" ""
+		(property "Digikey_Part_Number" "DMG2302UK-7DICT-ND"
 			(at 238.76 102.87 0)
 			(effects
@@
 			)
 		)
-		(property "Manufacturer_Product_Number" ""
+		(property "Manufacturer_Product_Number" "DMG2302UK-7"
 			(at 238.76 102.87 0)
 			(effects
@@
 			)
 		)
-		(property "Datasheet" "~"
+		(property "Datasheet" "https://www.digikey.ca/en/products/detail/yageo/RC1206FR-07470RL/728934"
 			(at 170.18 76.2 0)
 			(effects
@@
 			)
 		)
-		(property "Digikey_Part_Number" ""
+		(property "Digikey_Part_Number" "311-470FRCT-ND"
 			(at 170.18 76.2 90)
 			(effects
@@
 			)
 		)
-		(property "Manufacturer_Product_Number" ""
+		(property "Manufacturer_Product_Number" "RC1206FR-07470RL"
 			(at 170.18 76.2 90)
 			(effects
@@
 			)
 		)
-		(property "Datasheet" "~"
+		(property "Datasheet" "https://www.digikey.ca/en/products/detail/kemet/C1206C104J5RACTU/411249"
 			(at 67.31 105.41 0)
 			(effects
@@
 			)
 		)
-		(property "Digikey_Part_Number" ""
+		(property "Digikey_Part_Number" "399-C1206C104J5RACTUCT-ND"
 			(at 67.31 105.41 0)
 			(effects
@@
 			)
 		)
-		(property "Manufacturer_Product_Number" ""
+		(property "Manufacturer_Product_Number" "C1206C104J5RACTU"
 			(at 67.31 105.41 0)
 			(effects
@@
 			)
 		)
-		(property "Footprint" "BMS_footprints:SOT23_DMG230_DIO"
+		(property "Footprint" "TO-252-2"
 			(at 121.92 85.09 0)
 			(effects
@@
 			)
 		)
-		(property "Datasheet" "TO-252-2"
+		(property "Datasheet" "https://www.digikey.ca/en/products/detail/diodes-incorporated/ZXMN4A06KTC/991923?s=N4IgTCBcDaIFoA0CyA5ALAQQAwDYDSIAugL5A"
 			(at 121.92 85.09 0)
 			(effects
@@
 			)
 		)
-		(property "Digikey_Part_Number" ""
+		(property "Digikey_Part_Number" "31-ZXMN4A06KTCCT-ND"
 			(at 121.92 85.09 0)
 			(effects
@@
 			)
 		)
-		(property "Manufacturer_Product_Number" ""
+		(property "Manufacturer_Product_Number" "  ZXMN4A06KTC"
 			(at 121.92 85.09 0)
 			(effects
@@
 			)
 		)
-		(property "Datasheet" "~"
+		(property "Datasheet" "https://www.digikey.ca/en/products/detail/yageo/RC1206FR-07470RL/728934"
 			(at 53.34 80.01 0)
 			(effects
@@
 			)
 		)
-		(property "Digikey_Part_Number" ""
+		(property "Digikey_Part_Number" "311-470FRCT-ND"
 			(at 53.34 80.01 90)
 			(effects
@@
 			)
 		)
-		(property "Manufacturer_Product_Number" ""
+		(property "Manufacturer_Product_Number" "RC1206FR-07470RL"
 			(at 53.34 80.01 90)
 			(effects
@@
 			)
 		)
-		(property "Datasheet" "~"
+		(property "Datasheet" "https://www.digikey.ca/en/products/detail/kemet/C1206C104J5RACTU/411249"
 			(at 184.15 101.6 0)
 			(effects
@@
 			)
 		)
-		(property "Digikey_Part_Number" ""
+		(property "Digikey_Part_Number" "399-C1206C104J5RACTUCT-ND"
 			(at 184.15 101.6 0)
 			(effects
@@
 			)
 		)
-		(property "Manufacturer_Product_Number" ""
+		(property "Manufacturer_Product_Number" "C1206C104J5RACTU"
 			(at 184.15 101.6 0)
 			(effects
@@
 			)
 		)
-		(property "Datasheet" "~"
+		(property "Datasheet" "https://www.digikey.ca/en/products/detail/kemet/C1206C104J5RACTU/411249"
 			(at 176.53 101.6 0)
 			(effects
@@
 			)
 		)
-		(property "Digikey_Part_Number" ""
+		(property "Digikey_Part_Number" "399-C1206C104J5RACTUCT-ND"
 			(at 176.53 101.6 0)
 			(effects
@@
 			)
 		)
-		(property "Manufacturer_Product_Number" ""
+		(property "Manufacturer_Product_Number" "C1206C104J5RACTU"
 			(at 176.53 101.6 0)
 			(effects
@@
 			)
 		)
-		(property "Datasheet" "https://www.diodes.com/assets/Datasheets/DMG2302UK.pdf"
+		(property "Datasheet" "https://www.digikey.ca/en/products/detail/diodes-incorporated/DMG2302UK-7/6010142"
 			(at 238.76 81.28 0)
 			(effects
@@
 			)
 		)
-		(property "Digikey_Part_Number" ""
+		(property "Digikey_Part_Number" "DMG2302UK-7DICT-ND"
 			(at 238.76 81.28 0)
 			(effects
@@
 			)
 		)
-		(property "Manufacturer_Product_Number" ""
+		(property "Manufacturer_Product_Number" "DMG2302UK-7"
 			(at 238.76 81.28 0)
 			(effects
@@
 			)
 		)
-		(property "Datasheet" "~"
+		(property "Datasheet" "https://www.digikey.ca/en/products/detail/yageo/RC1206FR-07470RL/728934"
 			(at 170.18 90.17 0)
 			(effects
@@
 			)
 		)
-		(property "Digikey_Part_Number" ""
+		(property "Digikey_Part_Number" "311-470FRCT-ND"
 			(at 170.18 90.17 90)
 			(effects
@@
 			)
 		)
-		(property "Manufacturer_Product_Number" ""
+		(property "Manufacturer_Product_Number" "RC1206FR-07470RL"
 			(at 170.18 90.17 90)
 			(effects
@@
 			)
 		)
-		(property "Digikey_Part_Number" ""
+		(property "Digikey_Part_Number" "1662-S-8252AAG-M6T1UCT-ND"
 			(at 232.41 92.71 0)
 			(effects
@@
 			)
 		)
-		(property "Manufacturer_Product_Number" ""
+		(property "Manufacturer_Product_Number" "S-8252AAG-M6T1U"
 			(at 232.41 92.71 0)
 			(effects
